Commit message: Add nav2 stack

File: src/diff_drive/diffdrive_description/urdf/robot.urdf.xacro (robot description, xacro)
@@ -15,4 +15,5 @@
     <xacro:property name="caster_mass" value="0.10" />
     <xacro:property name="lidar_zoff" value="0.03" />
+    <xacro:arg name="use_3d_lidar" default="false"/>
     <link name="base_footprint" />
     <link name="base_link">
@@ -89,5 +90,5 @@
             <parameters>$(find diffdrive_bringup)/config/controllers.yaml</parameters>
             <ros>
-                <remapping>/diff_drive_controller/cmd_vel_unstamped:=/cmd_vel</remapping>
+                <remapping>/diff_drive_controller/cmd_vel:=/cmd_vel</remapping>
                 <remapping>/diff_drive_controller/odom:=/odom</remapping>
             </ros>
@@ -128,8 +129,26 @@
         <xacro:box_inertia m="0.1" w="0.1" d="0.1" h="0.1" />
     </link>
+    <link name="camera_link">
+        <visual>
+            <geometry>
+                <box size="0.05 0.1 0.05" />
+            </geometry>
+        </visual>
+        <collision>
+            <geometry>
+                <box size="0.05 0.1 0.05" />
+            </geometry>
+        </collision>
+        <xacro:box_inertia m="0.1" w="0.1" d="0.1" h="0.1" />
+    </link>
     <joint name="imu_joint" type="fixed">
         <parent link="base_link" />
         <child link="imu_link" />
         <origin xyz="0 0 0.01" />
+    </joint>
+    <joint name="camera_joint" type="fixed">
+        <parent link="imu_link" />
+        <child link="camera_link" />
+        <origin xyz="0 0 0.2" />
     </joint>
     <gazebo reference="imu_link">
@@ -161,4 +180,5 @@
     </joint>
     <gazebo reference="lidar_link">
+        <xacro:if value="$(arg use_3d_lidar)">
         <sensor name="RGLLidar" type="custom">
             <plugin filename="RGLServerPluginInstance" name="rgl::RGLServerPluginInstance">
@@ -182,4 +202,54 @@
             </plugin>
         </sensor>
+        </xacro:if>
+        <xacro:unless value="$(arg use_3d_lidar)">
+        <sensor name='gpu_lidar' type='gpu_lidar'>"
+            <gz_frame_id>base_link</gz_frame_id>
+            <topic>scan</topic>
+            <update_rate>10</update_rate>
+            <ray>
+                <scan>
+                    <horizontal>
+                        <samples>640</samples>
+                        <resolution>1</resolution>
+                        <min_angle>-1.396263</min_angle>
+                        <max_angle>1.396263</max_angle>
+                    </horizontal>
+                    <vertical>
+                        <samples>1</samples>
+                        <resolution>0.01</resolution>
+                        <min_angle>0</min_angle>
+                        <max_angle>0</max_angle>
+                    </vertical>
+                </scan>
+                <range>
+                    <min>0.08</min>
+                    <max>10.0</max>
+                    <resolution>0.01</resolution>
+                </range>
+            </ray>
+            <always_on>1</always_on>
+            <visualize>true</visualize>
+        </sensor>
+        </xacro:unless>
+    </gazebo>
+    <gazebo reference="camera_link">
+        <sensor name="depth_camera" type="depth_camera">
+            <gz_frame_id>camera_link</gz_frame_id>
+            <update_rate>10</update_rate>
+            <topic>depth_camera</topic>
+            <camera>
+                <horizontal_fov>1.05</horizontal_fov>
+                <image>
+                    <width>256</width>
+                    <height>256</height>
+                    <format>R_FLOAT32</format>
+                </image>
+                <clip>
+                    <near>0.1</near>
+                    <far>8.0</far>
+                </clip>
+            </camera>
+    </sensor>
     </gazebo>
 </robot>

Commit message: Add nav2 stack (#9)
* Add nav2 stack

* Add RMW_IMPLEMENTATION setup into devcontainer

* Update lidar params

* Fix RGLPLugin allow to use lidar_slam or nav2

File: src/diff_drive/diffdrive_description/urdf/robot.urdf.xacro (robot description, xacro)
@@ -15,4 +15,5 @@
     <xacro:property name="caster_mass" value="0.10" />
     <xacro:property name="lidar_zoff" value="0.03" />
+    <xacro:arg name="use_3d_lidar" default="false"/>
     <link name="base_footprint" />
     <link name="base_link">
@@ -89,5 +90,5 @@
             <parameters>$(find diffdrive_bringup)/config/controllers.yaml</parameters>
             <ros>
-                <remapping>/diff_drive_controller/cmd_vel_unstamped:=/cmd_vel</remapping>
+                <remapping>/diff_drive_controller/cmd_vel:=/cmd_vel</remapping>
                 <remapping>/diff_drive_controller/odom:=/odom</remapping>
             </ros>
@@ -128,8 +129,26 @@
         <xacro:box_inertia m="0.1" w="0.1" d="0.1" h="0.1" />
     </link>
+    <link name="camera_link">
+        <visual>
+            <geometry>
+                <box size="0.05 0.1 0.05" />
+            </geometry>
+        </visual>
+        <collision>
+            <geometry>
+                <box size="0.05 0.1 0.05" />
+            </geometry>
+        </collision>
+        <xacro:box_inertia m="0.1" w="0.1" d="0.1" h="0.1" />
+    </link>
     <joint name="imu_joint" type="fixed">
         <parent link="base_link" />
         <child link="imu_link" />
         <origin xyz="0 0 0.01" />
+    </joint>
+    <joint name="camera_joint" type="fixed">
+        <parent link="imu_link" />
+        <child link="camera_link" />
+        <origin xyz="0 0 0.2" />
     </joint>
     <gazebo reference="imu_link">
@@ -161,7 +180,11 @@
     </joint>
     <gazebo reference="lidar_link">
+        <xacro:if value="$(arg use_3d_lidar)">
         <sensor name="RGLLidar" type="custom">
             <plugin filename="RGLServerPluginInstance" name="rgl::RGLServerPluginInstance">
-                <range>245</range>
+                <range>245
+                    <min>0</min>
+                    <max>245</max>
+                </range>
                 <update_rate>20</update_rate>
                 <update_on_paused_sim>false</update_on_paused_sim>
@@ -182,4 +205,54 @@
             </plugin>
         </sensor>
+        </xacro:if>
+        <xacro:unless value="$(arg use_3d_lidar)">
+        <sensor name='gpu_lidar' type='gpu_lidar'>"
+            <gz_frame_id>base_link</gz_frame_id>
+            <topic>scan</topic>
+            <update_rate>10</update_rate>
+            <ray>
+                <scan>
+                    <horizontal>
+                        <samples>640</samples>
+                        <resolution>1</resolution>
+                        <min_angle>-2.4</min_angle>
+                        <max_angle>2.4</max_angle>
+                    </horizontal>
+                    <vertical>
+                        <samples>1</samples>
+                        <resolution>0.01</resolution>
+                        <min_angle>0</min_angle>
+                        <max_angle>0</max_angle>
+                    </vertical>
+                </scan>
+                <range>
+                    <min>0.08</min>
+                    <max>10.0</max>
+                    <resolution>0.01</resolution>
+                </range>
+            </ray>
+            <always_on>1</always_on>
+            <visualize>true</visualize>
+        </sensor>
+        </xacro:unless>
+    </gazebo>
+    <gazebo reference="camera_link">
+        <sensor name="depth_camera" type="depth_camera">
+            <gz_frame_id>camera_link</gz_frame_id>
+            <update_rate>10</update_rate>
+            <topic>depth_camera</topic>
+            <camera>
+                <horizontal_fov>1.05</horizontal_fov>
+                <image>
+                    <width>256</width>
+                    <height>256</height>
+                    <format>R_FLOAT32</format>
+                </image>
+                <clip>
+                    <near>0.1</near>
+                    <far>8.0</far>
+                </clip>
+            </camera>
+    </sensor>
     </gazebo>
 </robot>

Commit message: Add cameras to the model

File: src/diff_drive/diffdrive_description/urdf/robot.urdf.xacro (robot description, xacro)
@@ -129,5 +129,5 @@
         <xacro:box_inertia m="0.1" w="0.1" d="0.1" h="0.1" />
     </link>
-    <link name="camera_link">
+    <link name="camera_depth_link">
         <visual>
             <geometry>
@@ -138,4 +138,30 @@
             <geometry>
                 <box size="0.05 0.1 0.05" />
+            </geometry>
+        </collision>
+        <xacro:box_inertia m="0.1" w="0.1" d="0.1" h="0.1" />
+    </link>
+    <link name="right_camera_link">
+        <visual>
+            <geometry>
+                <box size="0.05 0.05 0.05" />
+            </geometry>
+        </visual>
+        <collision>
+            <geometry>
+                <box size="0.05 0.05 0.05" />
+            </geometry>
+        </collision>
+        <xacro:box_inertia m="0.1" w="0.1" d="0.1" h="0.1" />
+    </link>
+    <link name="left_camera_link">
+        <visual>
+            <geometry>
+                <box size="0.05 0.05 0.05" />
+            </geometry>
+        </visual>
+        <collision>
+            <geometry>
+                <box size="0.05 0.05 0.05" />
             </geometry>
         </collision>
@@ -147,8 +173,18 @@
         <origin xyz="0 0 0.01" />
     </joint>
-    <joint name="camera_joint" type="fixed">
+    <joint name="camera_depth_joint" type="fixed">
         <parent link="imu_link" />
-        <child link="camera_link" />
+        <child link="camera_depth_link" />
         <origin xyz="0 0 0.2" />
+    </joint>
+    <joint name="right_camera_joint" type="fixed">
+        <parent link="imu_link" />
+        <child link="right_camera_link" />
+        <origin xyz="0.1 -0.15 0.2" rpy="${-pi/2} 0 ${-pi/2}"/>
+    </joint>
+    <joint name="left_camera_joint" type="fixed">
+        <parent link="imu_link" />
+        <child link="left_camera_link" />
+        <origin xyz="0.1 0.15 0.2" rpy="${-pi/2} 0 ${-pi/2}"/>
     </joint>
     <gazebo reference="imu_link">
@@ -237,7 +273,7 @@
         </xacro:unless>
     </gazebo>
-    <gazebo reference="camera_link">
+    <gazebo reference="camera_depth_link">
         <sensor name="depth_camera" type="depth_camera">
-            <gz_frame_id>camera_link</gz_frame_id>
+            <gz_frame_id>camera_depth_link</gz_frame_id>
             <update_rate>10</update_rate>
             <topic>depth_camera</topic>
@@ -255,4 +291,32 @@
             </camera>
     </sensor>
+    <sensor name="right_camera" type="camera">
+        <always_on>true</always_on>
+        <visualize>true</visualize>
+        <update_rate>30</update_rate>
+        <topic>right_camera/image_raw</topic>
+        <gz_frame_id>right_camera_link</gz_frame_id>
+        <camera name="right_camera">
+            <image>
+                <width>1920</width>
+                <height>1080</height>
+            </image>
+            <camera_info_topic>right_camera/camera_info</camera_info_topic>
+        </camera>
+    </sensor>
+    <sensor name="left_camera" type="camera">
+        <always_on>true</always_on>
+        <visualize>true</visualize>
+        <update_rate>30</update_rate>
+        <topic>left_camera/image_raw</topic>
+        <gz_frame_id>left_camera_link</gz_frame_id>
+        <camera name="left_camera">
+            <image>
+                <width>1920</width>
+                <height>1080</height>
+            </image>
+            <camera_info_topic>left_camera/camera_info</camera_info_topic>
+        </camera>
+    </sensor>
     </gazebo>
 </robot>

Commit message: Update URDF and world config

File: src/diff_drive/diffdrive_description/urdf/robot.urdf.xacro (robot description, xacro)
@@ -181,10 +181,10 @@
         <parent link="imu_link" />
         <child link="right_camera_link" />
-        <origin xyz="0.1 -0.15 0.2" rpy="${-pi/2} 0 ${-pi/2}"/>
+        <origin xyz="0.1 -0.15 0.2" rpy="0 0 0"/>
     </joint>
     <joint name="left_camera_joint" type="fixed">
         <parent link="imu_link" />
         <child link="left_camera_link" />
-        <origin xyz="0.1 0.15 0.2" rpy="${-pi/2} 0 ${-pi/2}"/>
+        <origin xyz="0.1 0.15 0.2" rpy="0 0 0"/>
     </joint>
     <gazebo reference="imu_link">
@@ -295,5 +295,4 @@
     <sensor name="right_camera" type="camera">
         <always_on>true</always_on>
-        <visualize>true</visualize>
         <update_rate>20</update_rate>
         <topic>right_camera/image_raw</topic>
@@ -311,5 +310,4 @@
     <sensor name="left_camera" type="camera">
         <always_on>true</always_on>
-        <visualize>true</visualize>
         <update_rate>20</update_rate>
         <topic>left_camera/image_raw</topic>
